File: MM1_SRAM_64k_A.kicad_pcb (KiCad board)
At the start: 2 copper layers, 51.5 x 34 mm, 9 parts, among them J1 MM1_edgeConnector_5530843-2, U1 IS61LV256AL-10JL, U2 IS61LV256AL-10JL, U3 74AHC1G04, U4 74AHC1G32, U5 74AHC1G32

Commit message: custom SOJ-28 footprint and gerbert file
Parts:
- U1, U2: footprint Package_SO:SOIC-28W_7.5x17.9mm_P1.27mm -> SOJ28:SOJ-28_P1.27mm
Routing:
- net GND: track 88.2 -> 10.2 mm, vias 5 -> 2
- net /MEMADDRESS_11: track 28.2 -> 23.4 mm
- net /MEM1_~CE: track 30.7 -> 26.4 mm
- net /MEM_~WE: track 33.4 -> 30.5 mm
- net /MEMADDRESS_9: track 26.6 -> 24.0 mm, vias 1 -> 3
- net /MEM2_~CE: track 26.9 -> 29.5 mm
- net +3V3: track 51.3 -> 49.4 mm, vias 1 -> 2
- net /MEM_~CE: track 18.5 -> 20.1 mm
- net /MEMDATA_6: track 45.5 -> 44.2 mm
- net /MEMADDRESS_0: track 26.5 -> 27.7 mm
- net /MEMADDRESS_1: track 27.7 -> 26.6 mm
- net /MEMDATA_7: track 45.0 -> 44.1 mm
- net /MEMDATA_3: track 45.4 -> 44.5 mm
- net /MEMADDRESS_5: track 26.2 -> 25.3 mm
- net /MEM_~OE: track 43.0 -> 42.2 mm
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Other:
- net class Power added: clearance 0.2, trace_width 0.25, via_dia 0.45, via_drill 0.2
- net class Tension removed
- rule pad_to_mask_clearance: 0.2 -> 0
