File: MM1_SRAM_64k_A.sch (KiCad schematic (older format))
At the start: 9 parts, among them J1 MM1_edgeConnector_5530843-2, U1 IS61LV256AL-10JL, U2 IS61LV256AL-10JL, U3 74AHC1G04, U4 74AHC1G32, U5 74AHC1G32

Commit message: custom SOJ-28 footprint and gerbert file
Parts:
- U1, U2: footprint Package_SO:SOIC-28W_7.5x17.9mm_P1.27mm -> SOJ28:SOJ-28_P1.27mm
Changed lines of the file:
@@
 F 0 "U2" H 8300 4750 50  0000 C CNN
 F 1 "IS61LV256AL-10JL" H 8600 4650 50  0000 C CNN
-F 2 "Package_SO:SOIC-28W_7.5x17.9mm_P1.27mm" H 7700 4550 50  0001 C CNN
+F 2 "SOJ28:SOJ-28_P1.27mm" H 7700 4550 50  0001 C CNN
 F 3 "https://www.mouser.ch/datasheet/2/198/61LV256AL-258426.pdf" H 8200 3400 50  0001 C CNN
 	1    8200 3600
@@
 F 0 "U1" H 5600 4750 50  0000 C CNN
 F 1 "IS61LV256AL-10JL" H 5900 4650 50  0000 C CNN
-F 2 "Package_SO:SOIC-28W_7.5x17.9mm_P1.27mm" H 5000 4550 50  0001 C CNN
+F 2 "SOJ28:SOJ-28_P1.27mm" H 5000 4550 50  0001 C CNN
 F 3 "https://www.mouser.ch/datasheet/2/198/61LV256AL-258426.pdf" H 5500 3400 50  0001 C CNN
 	1    5500 3600
